Commit message: added world frame

File: urdf_creation/fr3.urdf (robot description, URDF)
Before this commit: robot fr3, 13 links, 12 joints
Links:
- added link world
Joints:
- added joint arm_to_world_fixed: type fixed, parent world, child fr3_link0, origin xyz=0 0 0 rpy=0 0 0
- joint fr3_hand_joint: origin xyz=0 0 0 rpy=0 0 -0.7853981633974483 -> xyz=0 0 0 rpy=0 0 -0.78539816339744830961566084581988
- joint fr3_joint2: origin xyz=0 0 0 rpy=-1.5707963267948966 0 0 -> xyz=0 0 0 rpy=-1.57079632679489661923132169163975 0 0
- joint fr3_joint3: origin xyz=0 -0.316 0 rpy=1.5707963267948966 0 0 -> xyz=0 -0.316 0 rpy=1.57079632679489661923132169163975 0 0
- joint fr3_joint4: origin xyz=0.0825 0 0 rpy=1.5707963267948966 0 0 -> xyz=0.0825 0 0 rpy=1.57079632679489661923132169163975 0 0
- joint fr3_joint5: origin xyz=-0.0825 0.384 0 rpy=-1.5707963267948966 0 0 -> xyz=-0.0825 0.384 0 rpy=-1.57079632679489661923132169163975 0 0
- joint fr3_joint6: origin xyz=0 0 0 rpy=1.5707963267948966 0 0 -> xyz=0 0 0 rpy=1.57079632679489661923132169163975 0 0
- joint fr3_joint7: origin xyz=0.088 0 0 rpy=1.5707963267948966 0 0 -> xyz=0.088 0 0 rpy=1.57079632679489661923132169163975 0 0

Commit message: tested pinocchio 3x (preview.) It delivers very accurate results, almost as accurate as from casadi_kin_dyn (which uses also pinocchio, but an older version.) TODO: compare casadi_kin_dyn with pinocchio 3 preview.

File: urdf_creation/fr3.urdf (robot description, URDF)
Before this commit: robot fr3, 14 links, 13 joints
Links:
- link fr3_hand: geometry collision mesh filename=/media/daten/Projekte/Studium/Master/Masterarbeit_SS2024/2D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; visual mesh filename=/media/daten/Projekte/Studium/Master/Masterarbeit_SS2024/2D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
- link fr3_leftfinger: geometry collision box size=17.5e-3 15.2e-3 18.5e-3; collision box size=17.5e-3 7e-3 23.5e-3
- link fr3_link0: geometry collision mesh filename=/media/daten/Projekte/Studium/Master/Masterarbeit_SS2024/2D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; visual mesh filename=/media/daten/Projekte/Studium/Master/Masterarbeit_SS2024/2D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
- link fr3_link1: geometry collision mesh filename=/media/daten/Projekte/Studium/Master/Masterarbeit_SS2024/2D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; visual mesh filename=/media/daten/Projekte/Studium/Master/Masterarbeit_SS2024/2D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
- link fr3_link2: geometry collision mesh filename=/media/daten/Projekte/Studium/Master/Masterarbeit_SS2024/2D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; visual mesh filename=/media/daten/Projekte/Studium/Master/Masterarbeit_SS2024/2D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
- link fr3_link3: geometry collision mesh filename=/media/daten/Projekte/Studium/Master/Masterarbeit_SS2024/2D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; visual mesh filename=/media/daten/Projekte/Studium/Master/Masterarbeit_SS2024/2D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
- link fr3_link4: geometry collision mesh filename=/media/daten/Projekte/Studium/Master/Masterarbeit_SS2024/2D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; visual mesh filename=/media/daten/Projekte/Studium/Master/Masterarbeit_SS2024/2D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
- link fr3_link5: geometry collision mesh filename=/media/daten/Projekte/Studium/Master/Masterarbeit_SS2024/2D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; visual mesh filename=/media/daten/Projekte/Studium/Master/Masterarbeit_SS2024/2D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
- link fr3_link6: geometry collision mesh filename=/media/daten/Projekte/Studium/Master/Masterarbeit_SS2024/2D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; visual mesh filename=/media/daten/Projekte/Studium/Master/Masterarbeit_SS2024/2D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
- link fr3_link7: geometry collision mesh filename=/media/daten/Projekte/Studium/Master/Masterarbeit_SS2024/2D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; visual mesh filename=/media/daten/Projekte/Studium/Master/Masterarbeit_SS2024/2D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
- link fr3_rightfinger: geometry collision box size=17.5e-3 15.2e-3 18.5e-3; collision box size=17.5e-3 7e-3 23.5e-3

Commit message: fixed bug with hand_tcp: now it have zero mass and zero inertia. Recreated matlab functions and matrices.

File: urdf_creation/fr3.urdf (robot description, URDF)
Before this commit: robot fr3, 14 links, 13 joints
Links:
- link fr3_hand_tcp: mass 1e-5 -> 0

Commit message: Reduced DOFs to 6. See notes in init_param_robot.m for updating to 7dof again.

File: urdf_creation/fr3.urdf (robot description, URDF)
Before this commit: robot fr3, 14 links, 13 joints
Joints:
- joint fr3_joint3: origin xyz=0 -0.316 0 rpy=1.57079632679489661923132169163975 0 0 -> xyz=0 -0.316 0 rpy=1.57079632679489661923132169163975 -0.78539816339744830961566084581988 0; type revolute -> fixed
