Commit message: removed robotic handle (1kg hand) and renamed file.

File: urdf_creation/ur5e.urdf (robot description, URDF)
Before this commit: robot ur5e_with_robotiq_hande, 14 links, 13 joints
Links:
- removed link base_link_inertia
- removed link flange
- removed link forearm_link
- removed link hand_e_link
- removed link hande_left_finger
- removed link hande_right_finger
- removed link shoulder_link
- removed link tool0
- removed link upper_arm_link
- removed link wrist_1_link
- removed link wrist_2_link
- removed link wrist_3_link
- added link ur5e_link0, mass 4.0; collision mesh filename=/media/daten/Projekte/Studium/Master/Masterarbeit_SS2024/2D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; visual mesh filename=/media/daten/Projekte/Studium/Master/Masterarbeit_SS2024/2D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
- added link ur5e_link1, mass 3.7; collision mesh filename=/media/daten/Projekte/Studium/Master/Masterarbeit_SS2024/2D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; visual mesh filename=/media/daten/Projekte/Studium/Master/Masterarbeit_SS2024/2D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
- added link ur5e_link2, mass 8.393; collision mesh filename=/media/daten/Projekte/Studium/Master/Masterarbeit_SS2024/2D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; visual mesh filename=/media/daten/Projekte/Studium/Master/Masterarbeit_SS2024/2D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
- added link ur5e_link3, mass 2.275; collision mesh filename=/media/daten/Projekte/Studium/Master/Masterarbeit_SS2024/2D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; visual mesh filename=/media/daten/Projekte/Studium/Master/Masterarbeit_SS2024/2D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
- added link ur5e_link4, mass 1.219; collision mesh filename=/media/daten/Projekte/Studium/Master/Masterarbeit_SS2024/2D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; visual mesh filename=/media/daten/Projekte/Studium/Master/Masterarbeit_SS2024/2D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
- added link ur5e_link5, mass 1.219; collision mesh filename=/media/daten/Projekte/Studium/Master/Masterarbeit_SS2024/2D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; visual mesh filename=/media/daten/Projekte/Studium/Master/Masterarbeit_SS2024/2D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
- added link ur5e_link6, mass 0.1879; collision mesh filename=/media/daten/Projekte/Studium/Master/Masterarbeit_SS2024/2D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; visual mesh filename=/media/daten/Projekte/Studium/Master/Masterarbeit_SS2024/2D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
Joints:
- removed joint base_link-base_link_inertia
- removed joint elbow_joint
- removed joint flange-tool0
- removed joint hande_left_finger_joint
- removed joint hande_right_finger_joint
- removed joint robotiq_hande_base_joint
- removed joint shoulder_lift_joint
- removed joint shoulder_pan_joint
- removed joint wrist_1_joint
- removed joint wrist_2_joint
- removed joint wrist_3-flange
- removed joint wrist_3_joint
- added joint basejoint: type fixed, parent base_link, child ur5e_link0, origin xyz=0 0 0 rpy=0 0 3.14159265359
- added joint ur5e_joint1: type revolute, parent ur5e_link0, child ur5e_link1, origin xyz=0 0 0.1625 rpy=0 0 0, axis 0 0 1, limit lower=-6.28318530718 upper=6.28318530718 effort=150.0 velocity=3.14159265359
- added joint ur5e_joint2: type revolute, parent ur5e_link1, child ur5e_link2, origin xyz=0 0 0 rpy=1.570796327 0 0, axis 0 0 1, limit lower=-6.28318530718 upper=6.28318530718 effort=150.0 velocity=3.14159265359
- added joint ur5e_joint3: type revolute, parent ur5e_link2, child ur5e_link3, origin xyz=-0.425 0 0 rpy=0 0 0, axis 0 0 1, limit lower=-3.14159265359 upper=3.14159265359 effort=150.0 velocity=3.14159265359
- added joint ur5e_joint4: type revolute, parent ur5e_link3, child ur5e_link4, origin xyz=-0.3922 0 0.1333 rpy=0 0 0, axis 0 0 1, limit lower=-6.28318530718 upper=6.28318530718 effort=28.0 velocity=3.14159265359
- added joint ur5e_joint5: type revolute, parent ur5e_link4, child ur5e_link5, origin xyz=0 -0.0997 -2.0448811823e-11 rpy=1.570796327 0 0, axis 0 0 1, limit lower=-6.28318530718 upper=6.28318530718 effort=28.0 velocity=3.14159265359
- added joint ur5e_joint6: type revolute, parent ur5e_link5, child ur5e_link6, origin xyz=0 0.0996 -2.04283014801e-11 rpy=1.57079632659 3.14159265359 3.14159265359, axis 0 0 1, limit lower=-6.28318530718 upper=6.28318530718 effort=28.0 velocity=3.14159265359

Commit message: Added ur5e Models - Simulink Model - Mujoco Model - Visual files for Simulink - urdf file with corrections

File: urdf_creation/ur5e.urdf (robot description, URDF)
Before this commit: robot ur5e_robot, 9 links, 8 joints
Links:
- removed link ur5e_link0
- added link ur5e_tcp, mass 0.1; collision box size=0.01 0.01 0.01
- link base_link: mass None -> 4.0; geometry collision mesh filename=collision_base.stl; visual mesh filename=ur5e-link0_con.stl
- link ur5e_link1: geometry collision mesh filename=collision_shoulder.stl; visual mesh filename=ur5e-link1_cap.stl
- link ur5e_link2: geometry collision mesh filename=collision_upperarm.stl; visual mesh filename=ur5e-link2_cap1.stl
- link ur5e_link3: geometry collision mesh filename=collision_forearm.stl; visual mesh filename=ur5e-link3_cap.stl
- link ur5e_link4: geometry collision mesh filename=collision_wrist1.stl; visual mesh filename=ur5e-link4_cap.stl
- link ur5e_link5: geometry collision mesh filename=collision_wrist2.stl; visual mesh filename=ur5e-link5_cap.stl
- link ur5e_link6: geometry collision mesh filename=collision_wrist3.stl; visual mesh filename=ur5e-link6_rod.stl
Joints:
- removed joint basejoint
- added joint TCP_fixed_joint: type fixed, parent ur5e_link6, child ur5e_tcp, origin xyz=0.0 0.1 0.0 rpy=0.0 0.0 1.57079632679
- joint ur5e_joint1: origin xyz=0 0 0.1625 rpy=0 0 0 -> xyz=0.0 0.0 0.1625 rpy=0.0 0.0 0.0; parent ur5e_link0 -> base_link
- joint ur5e_joint2: axis 0 0 1 -> 0 1 0; origin xyz=0 0 0 rpy=1.570796327 0 0 -> xyz=0.0 0.138 0.0 rpy=0.0 1.57079632679 0.0
- joint ur5e_joint3: axis 0 0 1 -> 0 1 0; limit lower=-3.14159265359 upper=3.14159265359 effort=150.0 velocity=3.14159265359 -> lower=-6.28318530718 upper=6.28318530718 effort=150.0 velocity=3.14159265359; origin xyz=-0.425 0 0 rpy=0 0 0 -> xyz=0.0 -0.131 0.425 rpy=0.0 0.0 0.0
- joint ur5e_joint4: axis 0 0 1 -> 0 1 0; limit lower=-6.28318530718 upper=6.28318530718 effort=28.0 velocity=3.14159265359 -> lower=-6.28318530718 upper=6.28318530718 effort=28.0 velocity=6.28; origin xyz=-0.3922 0 0.1333 rpy=0 0 0 -> xyz=0.0 0.0 0.392 rpy=0.0 1.57079632679 0.0
- joint ur5e_joint5: limit lower=-6.28318530718 upper=6.28318530718 effort=28.0 velocity=3.14159265359 -> lower=-6.28318530718 upper=6.28318530718 effort=28.0 velocity=6.28; origin xyz=0 -0.0997 -2.0448811823e-11 rpy=1.570796327 0 0 -> xyz=0.0 0.127 0.0 rpy=0.0 0.0 0.0
- joint ur5e_joint6: axis 0 0 1 -> 0 1 0; limit lower=-6.28318530718 upper=6.28318530718 effort=28.0 velocity=3.14159265359 -> lower=-6.28318530718 upper=6.28318530718 effort=28.0 velocity=6.28; origin xyz=0 0.0996 -2.04283014801e-11 rpy=1.57079632659 3.14159265359 3.14159265359 -> xyz=0.0 0.0 0.1 rpy=0.0 0.0 0.0

Commit message: fixed bug in ur5e model: tcp had useless rotation. Also some lengths wasn't correct. forward kinematics is now correct, but all trajectories has changed now!
- fixed refsys mpc for kinetic model.

File: urdf_creation/ur5e.urdf (robot description, URDF)
Before this commit: robot ur5e_robot, 9 links, 8 joints
Joints:
- joint TCP_fixed_joint: origin xyz=0.0 0.1 0.0 rpy=0.0 0.0 1.57079632679 -> xyz=0.0 0.0996 0.0 rpy=0.0 0.0 0.0
- joint ur5e_joint4: origin xyz=0.0 0.0 0.392 rpy=0.0 1.57079632679 0.0 -> xyz=0.0 0.0 0.3922 rpy=0.0 1.57079632679 0.0
- joint ur5e_joint6: origin xyz=0.0 0.0 0.1 rpy=0.0 0.0 0.0 -> xyz=0.0 0.0 0.0997 rpy=0.0 0.0 0.0
