Commit message: deleted mass from link8

File: urdf_creation/fr3_no_hand_6dof.urdf (robot description, URDF)
Before this commit: robot fr3, 11 links, 10 joints
Links:
- link fr3_link8: mass 1e-5 -> 0

Commit message: - compared urdf files they are equals - in matlab pinocchio and meshcat differ in 1e-15 - added s functions to realtime franka software but didn't test it.

File: urdf_creation/fr3_no_hand_6dof.urdf (robot description, URDF)
Before this commit: robot fr3, 11 links, 10 joints
Links:
- link fr3_link0: geometry collision mesh filename=collision/link0.stl; visual mesh filename=visual/link0.obj
- link fr3_link1: geometry collision mesh filename=collision/link1.stl; visual mesh filename=visual/link1.obj
- link fr3_link2: geometry collision mesh filename=collision/link2.stl; visual mesh filename=visual/link2.obj
- link fr3_link3: geometry collision mesh filename=collision/link3.stl; visual mesh filename=visual/link3.obj
- link fr3_link4: geometry collision mesh filename=collision/link4.stl; visual mesh filename=visual/link4.obj
- link fr3_link5: geometry collision mesh filename=collision/link5.stl; visual mesh filename=visual/link5.obj
- link fr3_link6: geometry collision mesh filename=collision/link6.stl; visual mesh filename=visual/link6.obj
- link fr3_link7: geometry collision mesh filename=collision/link7.stl; visual mesh filename=visual/link7.obj
