Commit message: - for a real system is it not a good idea to force a joint to a fixed value because it is not ensured that this joint will always have this value. Therefore I use the full 7dof model (without hand tcp) and implement a joint space controller with a high stiffness to force the fixed joint position. This have the advantage, that all dynamic matrices are correct because they also contains the current "fixed" joint value.

File: urdf_creation/fr3_no_hand_7dof.urdf (robot description, URDF)
Before this commit: robot fr3, 11 links, 10 joints
Joints:
- joint fr3_joint3: type fixed -> revolute

Commit message: removed unneded includes and added a script for running xml files in mujoco.

File: urdf_creation/fr3_no_hand_7dof.urdf (robot description, URDF)
Before this commit: robot fr3, 11 links, 10 joints
Joints:
- joint fr3_link8_tcp_joint: origin xyz=0 0 0 rpy=0 0 0 -> xyz=0 0 0 rpy=0 0 -0.78539816339744830961566084581988
